File: SensitiveSole.kicad_pcb (KiCad board)
At the start: 2 copper layers, 33 x 33 mm, 7 parts, among them J1 DF12-36NOLEGS-FEMALE, J3 DF12-36NOLEGS-MALE

Commit message: update
Parts:
- added C1: 0.1µ, Capacitor_SMD:C_0603_1608Metric_Pad1.08x0.95mm_HandSolder, F.Cu at (204.3, 58.2)
- added C2: 10µ, Capacitor_SMD:C_0603_1608Metric_Pad1.08x0.95mm_HandSolder, F.Cu at (204.3, 60.7)
- added J1: Conn_01x24, Connector_FFC-FPC:Molex_200528-0240_1x24-1MP_P1.00mm_Horizontal, F.Cu at (143.2, 119.3)
- added R1: 10k, Resistor_SMD:R_0603_1608Metric_Pad0.98x0.95mm_HandSolder, F.Cu at (171.0, 112.5)
- added R10: 10k, Resistor_SMD:R_0603_1608Metric_Pad0.98x0.95mm_HandSolder, F.Cu at (207.7, 90.2)
- added R11: 10k, Resistor_SMD:R_0603_1608Metric_Pad0.98x0.95mm_HandSolder, F.Cu at (207.7, 92.7)
- added R12: 10k, Resistor_SMD:R_0603_1608Metric_Pad0.98x0.95mm_HandSolder, F.Cu at (212.0, 82.7)
- added R13: 10k, Resistor_SMD:R_0603_1608Metric_Pad0.98x0.95mm_HandSolder, F.Cu at (212.0, 85.2)
- added R14: 10k, Resistor_SMD:R_0603_1608Metric_Pad0.98x0.95mm_HandSolder, F.Cu at (212.0, 87.7)
- added R15: 10k, Resistor_SMD:R_0603_1608Metric_Pad0.98x0.95mm_HandSolder, F.Cu at (212.0, 90.2)
- added R16: 10k, Resistor_SMD:R_0603_1608Metric_Pad0.98x0.95mm_HandSolder, F.Cu at (212.0, 92.7)
- added R2: 10k, Resistor_SMD:R_0603_1608Metric_Pad0.98x0.95mm_HandSolder, F.Cu at (203.3, 82.7)
- added R3: 10k, Resistor_SMD:R_0603_1608Metric_Pad0.98x0.95mm_HandSolder, F.Cu at (203.3, 85.2)
- added R4: 10k, Resistor_SMD:R_0603_1608Metric_Pad0.98x0.95mm_HandSolder, F.Cu at (203.3, 87.7)
- added R5: 10k, Resistor_SMD:R_0603_1608Metric_Pad0.98x0.95mm_HandSolder, F.Cu at (203.3, 90.2)
- added R6: 10k, Resistor_SMD:R_0603_1608Metric_Pad0.98x0.95mm_HandSolder, F.Cu at (203.3, 92.7)
- added R7: 10k, Resistor_SMD:R_0603_1608Metric_Pad0.98x0.95mm_HandSolder, F.Cu at (207.7, 82.7)
- added R8: 10k, Resistor_SMD:R_0603_1608Metric_Pad0.98x0.95mm_HandSolder, F.Cu at (207.7, 85.2)
- added R9: 10k, Resistor_SMD:R_0603_1608Metric_Pad0.98x0.95mm_HandSolder, F.Cu at (207.7, 87.7)
- added U1: CD74HC4067SM, Package_SO:SSOP-24_5.3x8.2mm_P0.65mm, F.Cu at (183.9, 74.1)
- added U2: CD74HC4067SM, Package_SO:SSOP-24_5.3x8.2mm_P0.65mm, F.Cu at (183.9, 97.5)
- renumbered J3 to BOTTOM_DF12, J1 to TOP_DF12
Connections:
- net /ADC renamed /IO38
- BOTTOM_DF12 pad 1: Net-(J3-Pad1) -> /IO36
- BOTTOM_DF12 pad 10: Net-(J3-Pad10) -> /PB
- BOTTOM_DF12 pad 11: Net-(J3-Pad11) -> /IO35
- BOTTOM_DF12 pad 12: Net-(J3-Pad12) -> /RESET
- BOTTOM_DF12 pad 13: Net-(J3-Pad13) -> /IO32
- BOTTOM_DF12 pad 14: Net-(J3-Pad14) -> /GPIO0
- BOTTOM_DF12 pad 15: Net-(J3-Pad15) -> /IO33
- BOTTOM_DF12 pad 16: Net-(J3-Pad16) -> /RXD
- BOTTOM_DF12 pad 17: Net-(J3-Pad17) -> /IO25
- BOTTOM_DF12 pad 18: Net-(J3-Pad18) -> /TXD
- BOTTOM_DF12 pad 19: Net-(J3-Pad19) -> /IO26
- BOTTOM_DF12 pad 2: Net-(J3-Pad2) -> +5V
- BOTTOM_DF12 pad 20: Net-(J3-Pad20) -> /SCK
- BOTTOM_DF12 pad 21: Net-(J3-Pad21) -> /IO27
- BOTTOM_DF12 pad 22: Net-(J3-Pad22) -> /MOSI
- BOTTOM_DF12 pad 23: Net-(J3-Pad23) -> /IO14
- BOTTOM_DF12 pad 24: Net-(J3-Pad24) -> /MISO
- BOTTOM_DF12 pad 25: Net-(J3-Pad25) -> /IO15
- BOTTOM_DF12 pad 26: Net-(J3-Pad26) -> /SDA
- BOTTOM_DF12 pad 27: Net-(J3-Pad27) -> /IO12
- BOTTOM_DF12 pad 28: Net-(J3-Pad28) -> /SCL
- BOTTOM_DF12 pad 29: Net-(J3-Pad29) -> /IO13
- BOTTOM_DF12 pad 30: Net-(J3-Pad30) -> +3.3V
- BOTTOM_DF12 pad 31: Net-(J3-Pad31) -> /IO4
- BOTTOM_DF12 pad 32: VCC -> +3.3V
- BOTTOM_DF12 pad 33: Net-(J3-Pad33) -> /IO5
- BOTTOM_DF12 pad 35: Net-(J3-Pad35) -> /GPIO2
- BOTTOM_DF12 pad 4: Net-(J3-Pad4) -> +5V
- BOTTOM_DF12 pad 5: Net-(J3-Pad5) -> /IO39
- BOTTOM_DF12 pad 6: Net-(J3-Pad6) -> /BATT
- BOTTOM_DF12 pad 7: Net-(J3-Pad7) -> /IO34
- BOTTOM_DF12 pad 8: Net-(J3-Pad8) -> /VBATT
- BOTTOM_DF12 pad 9: Net-(J3-Pad9) -> /IO37
- TOP_DF12 pad 1: Net-(J1-Pad1) -> +5V
- TOP_DF12 pad 10: Net-(J1-Pad10) -> /IO37
- TOP_DF12 pad 11: Net-(J1-Pad11) -> /RESET
- TOP_DF12 pad 12: Net-(J1-Pad12) -> /IO35
- TOP_DF12 pad 13: Net-(J1-Pad13) -> /GPIO0
- TOP_DF12 pad 14: Net-(J1-Pad14) -> /IO32
- TOP_DF12 pad 15: Net-(J1-Pad15) -> /RXD
- TOP_DF12 pad 16: Net-(J1-Pad16) -> /IO33
- TOP_DF12 pad 17: Net-(J1-Pad17) -> /TXD
- TOP_DF12 pad 18: Net-(J1-Pad18) -> /IO25
- TOP_DF12 pad 19: Net-(J1-Pad19) -> /SCK
- TOP_DF12 pad 2: Net-(J1-Pad2) -> /IO36
- TOP_DF12 pad 20: Net-(J1-Pad20) -> /IO26
- TOP_DF12 pad 21: Net-(J1-Pad21) -> /MOSI
- TOP_DF12 pad 22: Net-(J1-Pad22) -> /IO27
- TOP_DF12 pad 23: Net-(J1-Pad23) -> /MISO
- TOP_DF12 pad 24: Net-(J1-Pad24) -> /IO14
- TOP_DF12 pad 25: Net-(J1-Pad25) -> /SDA
- TOP_DF12 pad 26: Net-(J1-Pad26) -> /IO15
- TOP_DF12 pad 27: Net-(J1-Pad27) -> /SCL
- TOP_DF12 pad 28: Net-(J1-Pad28) -> /IO12
- TOP_DF12 pad 29: Net-(J1-Pad29) -> +3.3V
- TOP_DF12 pad 3: Net-(J1-Pad3) -> +5V
- TOP_DF12 pad 30: Net-(J1-Pad30) -> /IO13
- TOP_DF12 pad 31: VCC -> +3.3V
- TOP_DF12 pad 32: Net-(J1-Pad32) -> /IO4
- TOP_DF12 pad 34: Net-(J1-Pad34) -> /IO5
- TOP_DF12 pad 36: Net-(J1-Pad36) -> /GPIO2
- TOP_DF12 pad 5: Net-(J1-Pad5) -> /BATT
- TOP_DF12 pad 6: Net-(J1-Pad6) -> /IO39
- TOP_DF12 pad 7: Net-(J1-Pad7) -> /VBATT
- TOP_DF12 pad 8: Net-(J1-Pad8) -> /IO34
- TOP_DF12 pad 9: Net-(J1-Pad9) -> /PB
Routing:
- net (no net): vias 1 -> 0
