File: SensitiveSole.kicad_pcb (KiCad board)
At the start: 2 copper layers, 33 x 33 mm, 28 parts, among them J1 Conn_01x24, U1 CD74HC4067SM, U2 CD74HC4067SM

Commit message: doc
Parts:
- moved U1 13.0 mm to (175.2, 83.8)
Changed lines of the file:
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@@
   )
   (footprint "Package_SO:SSOP-24_5.3x8.2mm_P0.65mm" (layer "F.Cu")
-    (at 183.9 74.125)
+    (at 175.216 83.801)
     (descr "24-Lead Plastic Shrink Small Outline (SS)-5.30 mm Body [SSOP] (see Microchip Packaging Specification 00000049BS.pdf)")
     (tags "SSOP 0.65")

Commit message: base clean
Parts:
- removed R10, R11, R12, R13, R14, R15, R16, R8, R9: 10k, Resistor_SMD:R_0603_1608Metric_Pad0.98x0.95mm_HandSolder
- removed TOP_DF12: DF12-36NOLEGS-FEMALE, MovuinoESP8266:DF12-36-DP-NL-noPad
- moved C1 74.7 mm to (180.6, 129.0), turned to 90 degrees
- moved C2 71.5 mm to (183.1, 129.0), turned to 90 degrees
- moved R7 65.7 mm to (143.7, 97.4)
- moved R5 59.7 mm to (143.7, 92.1)
- moved R6 59.7 mm to (143.7, 94.4)
- moved R2 56.6 mm to (147.7, 92.9)
- moved R3 56.5 mm to (147.7, 95.1)
- moved R4 56.5 mm to (147.7, 97.4)
- moved U2 55.0 mm to (129.0, 95.5)
- moved U1 47.0 mm to (139.6, 114.4), turned to -90 degrees
- moved R1 32.0 mm to (147.7, 90.6)
- moved FPC1 17.0 mm to (136.5, 103.6)
- moved U$8 12.6 mm to (135.2, 104.1)
- moved ? 11.3 mm to (151.0, 118.0)
- moved ? 11.3 mm to (122.0, 89.0)
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- renumbered J1 to FPC1
Connections:
- BOTTOM_DF12 pad 1: /IO36 -> unconnected-(BOTTOM_DF12-Pad1)
- BOTTOM_DF12 pad 11: /IO35 -> unconnected-(BOTTOM_DF12-Pad11)
- BOTTOM_DF12 pad 25: /IO15 -> unconnected-(BOTTOM_DF12-Pad25)
- BOTTOM_DF12 pad 29: /IO13 -> unconnected-(BOTTOM_DF12-Pad29)
- BOTTOM_DF12 pad 3: /IO38 -> unconnected-(BOTTOM_DF12-Pad3)
- BOTTOM_DF12 pad 31: /IO4 -> unconnected-(BOTTOM_DF12-Pad31)
- BOTTOM_DF12 pad 35: /GPIO2 -> /IO2
- BOTTOM_DF12 pad 7: /IO34 -> unconnected-(BOTTOM_DF12-Pad7)
- BOTTOM_DF12 pad 9: /IO37 -> unconnected-(BOTTOM_DF12-Pad9)
- FPC1 pad 10: unconnected-(J1-Pin_10-Pad10) -> /ROW8
- FPC1 pad 11: unconnected-(J1-Pin_11-Pad11) -> /ROW9
- FPC1 pad 12: unconnected-(J1-Pin_12-Pad12) -> /ROW10
- FPC1 pad 13: unconnected-(J1-Pin_13-Pad13) -> /ROW11
- FPC1 pad 14: unconnected-(J1-Pin_14-Pad14) -> /ROW12
- FPC1 pad 15: unconnected-(J1-Pin_15-Pad15) -> /ROW13
- FPC1 pad 16: unconnected-(J1-Pin_16-Pad16) -> /ROW14
- FPC1 pad 17: unconnected-(J1-Pin_17-Pad17) -> /COL6
- FPC1 pad 18: unconnected-(J1-Pin_18-Pad18) -> /COL5
- FPC1 pad 19: unconnected-(J1-Pin_19-Pad19) -> /COL4
- FPC1 pad 2: unconnected-(J1-Pin_2-Pad2) -> /ROW0
- FPC1 pad 20: unconnected-(J1-Pin_20-Pad20) -> /COL3
- FPC1 pad 21: unconnected-(J1-Pin_21-Pad21) -> /COL2
- FPC1 pad 22: unconnected-(J1-Pin_22-Pad22) -> /COL1
- FPC1 pad 23: unconnected-(J1-Pin_23-Pad23) -> /COL0
- FPC1 pad 3: unconnected-(J1-Pin_3-Pad3) -> /ROW1
- FPC1 pad 4: unconnected-(J1-Pin_4-Pad4) -> /ROW2
- FPC1 pad 5: unconnected-(J1-Pin_5-Pad5) -> /ROW3
- FPC1 pad 6: unconnected-(J1-Pin_6-Pad6) -> /ROW4
- FPC1 pad 7: unconnected-(J1-Pin_7-Pad7) -> /ROW5
- FPC1 pad 8: unconnected-(J1-Pin_8-Pad8) -> /ROW6
- FPC1 pad 9: unconnected-(J1-Pin_9-Pad9) -> /ROW7
- U1 pad 1: /IO25 -> /IO39
- U1 pad 10: /IO33 -> /IO32
- U1 pad 11: /IO32 -> /IO33
- U1 pad 13: /IO27 -> /IO26
- U1 pad 14: /IO26 -> /IO25
- U1 pad 16: /COL15 -> unconnected-(U1-I15-Pad16)
- U1 pad 17: /COL14 -> unconnected-(U1-I14-Pad17)
- U1 pad 18: /COL13 -> unconnected-(U1-I13-Pad18)
- U1 pad 19: /COL12 -> unconnected-(U1-I12-Pad19)
- U1 pad 2: /COL7 -> unconnected-(U1-I7-Pad2)
- U1 pad 20: /COL11 -> unconnected-(U1-I11-Pad20)
- U1 pad 21: /COL10 -> unconnected-(U1-I10-Pad21)
- U1 pad 22: /COL9 -> unconnected-(U1-I9-Pad22)
- U1 pad 23: /COL8 -> unconnected-(U1-I8-Pad23)
- U2 pad 1: /IO12 -> /IO2
- U2 pad 10: /IO13 -> /IO27
- U2 pad 11: /IO4 -> /IO14
- U2 pad 13: /IO14 -> /IO5
- U2 pad 14: /IO15 -> /IO12
- U2 pad 16: /ROW15 -> unconnected-(U2-I15-Pad16)
Routing:
- net GND: track 4.25 -> 0.50 mm
- net +5V: track 0.00 -> 0.50 mm
- net +3.3V: track 0.00 -> 0.50 mm

Commit message: v0.99
Parts:
- added C3: 0.1µ, Capacitor_SMD:C_0603_1608Metric_Pad1.08x0.95mm_HandSolder, B.Cu at (143.6, 90.9)
- added D1: SK6812, LED_SMD:LED_SK6812_PLCC4_5.0x5.0mm_P3.2mm, F.Cu at (136.5, 94.3)
- added R8: 470, Resistor_SMD:R_0603_1608Metric_Pad0.98x0.95mm_HandSolder, B.Cu at (128.6, 105.2)
- C1, C2, R1, R2, R3, R4, R5, R6, R7, U1, U2: moved to B.Cu
- moved C2 63.0 mm to (122.4, 112.2), turned to -90 degrees
- moved C1 58.1 mm to (124.9, 112.2), turned to -90 degrees
- moved U$8 28.5 mm to (113.4, 85.8)
- moved R1 24.1 mm to (145.0, 114.5), turned to 180 degrees
- moved R2 20.6 mm to (148.5, 113.4), turned to 180 degrees
- moved R5 18.0 mm to (145.0, 110.0), turned to 180 degrees
- moved R3 17.4 mm to (145.0, 112.3), turned to 180 degrees
- moved R6 15.4 mm to (148.5, 108.9), turned to 180 degrees
- moved R4 13.8 mm to (148.5, 111.2), turned to 180 degrees
- moved R7 10.5 mm to (145.0, 107.8), turned to 180 degrees
- moved U2 7.58 mm to (136.5, 94.5)
- moved U1 6.75 mm to (133.5, 111.5), turned to 180 degrees
Connections:
- BOTTOM_DF12 pad 25: unconnected-(BOTTOM_DF12-Pad25) -> /IO15
Routing:
- net +3.3V: track 0.50 -> 73.1 mm, vias 0 -> 4
- net Net-(D1-DIN): track 0.00 -> 36.9 mm, vias 0 -> 1
- net /IO5: track 0.00 -> 36.5 mm
- net /IO12: track 0.00 -> 34.3 mm
- net /IO2: track 0.00 -> 27.6 mm, vias 0 -> 2
- net /COL1: track 0.00 -> 24.5 mm, vias 0 -> 1
- net /IO26: track 0.00 -> 24.2 mm
- net /COL0: track 0.00 -> 23.9 mm, vias 0 -> 1
- net /IO25: track 0.00 -> 22.7 mm
- net /IO14: track 0.00 -> 22.6 mm
- net /IO27: track 0.00 -> 21.1 mm
- net /IO33: track 0.00 -> 20.9 mm
- net /IO32: track 0.00 -> 20.8 mm
- net /COL3: track 0.00 -> 20.0 mm, vias 0 -> 1
- net /ROW14: track 0.00 -> 18.6 mm, vias 0 -> 1
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- added copper zone on B.Cu, net GND
- added copper zone on F.Cu, net GND

Commit message: graphism
Parts:
- 0: renamed from R1; value 10k -> 10kΩ
- moved U$8 36.2 mm to (136.5, 113.7)
- moved C1 0.60 mm to (125.5, 112.2)
- moved C2 0.20 mm to (122.2, 112.2)
- renumbered C3 to 0, R2 to 1, R3 to 2, R4 to 3, R5 to 4, R6 to 5, R7 to 6, U1 to COLS, U2 to ROWS
Routing:
- net GND: track 12.0 -> 32.2 mm
- net +3.3V: track 73.1 -> 72.1 mm
- net /COL3: track 20.0 -> 19.0 mm
- net /IO5: track 36.5 -> 35.7 mm
- net /ROW6: track 7.42 -> 8.16 mm
- net /ROW7: track 7.15 -> 7.88 mm
- net /IO12: track 34.3 -> 33.6 mm
Other:
- board text added: "Adrien Husson"
- board text added: "Sensitive Sole v2.0"

Commit message: update
Parts:
- BOTTOM_DF12: footprint MovuinoESP8266:DF12-36-DP-NL -> Movuino:DF12-36-DP-NL
Other:
- board text added: "Adrn Hssn"
- board text removed: "Adrien Husson"
Changed lines of the file:
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@@
     (pad "" np_thru_hole circle (at 29 0) (size 2.1 2.1) (drill 2) (layers "*.Cu" "B.Mask"))
   )
-  (footprint "MovuinoESP8266:DF12-36-DP-NL" (layer "B.Cu")
+  (footprint "Movuino:DF12-36-DP-NL" (layer "B.Cu")
     (at 123.500014 103.499986 -90)
     (descr "Hirose DF12 Pattern with metal fitting, 32 positions")
@@
     (property "Sheetname" "")
     (attr through_hole)
-    (fp_text reference "BOTTOM_DF12" (at 2.5 13 90) (layer "B.SilkS") hide
+    (fp_text reference "BOTTOM_DF12" (at 0 0 90) (layer "B.SilkS") hide
         (effects (font (size 0.60325 0.60325) (thickness 0.0508)) (justify right top mirror))
     )
-    (fp_text value "DF12-36NOLEGS-MALE" (at 7.5 18.5 90) (layer "B.SilkS") hide
+    (fp_text value "DF12-36NOLEGS-MALE" (at 0 0 90) (layer "B.SilkS") hide
         (effects (font (size 1.27 1.27) (thickness 0.15)) (justify right top mirror))
     )
@@
       )
       (stroke (width 0) (type solid)) (fill solid) (layer "B.Fab"))
-    (pad "" np_thru_hole circle (at -5.3 1.5 270) (size 0.7 0.7) (drill 0.7) (layers "F&B.Cu" "*.Mask"))
+    (pad "" np_thru_hole circle (at -5.3 1.5 270) (size 0.7 0.7) (drill 0.7) (layers "*.Cu" "*.Mask"))
     (pad "" np_thru_hole circle (at 5.3 1.5 270) (size 0.7 0.7) (drill 0.7) (layers "*.Cu" "*.Mask"))
     (pad "1" smd rect (at -4.25 -1.8001 270) (size 0.3 1.6) (layers "B.Cu" "B.Mask")
@@
         (effects (font (size 1 1) (thickness 0.15)) (justify mirror))
     )
-    (fp_text value "10kΩ" (at -1.558 -2.64) (layer "B.Fab")
+    (fp_text value "10kΩ" (at -1.558 9.11) (layer "B.Fab")
         (effects (font (size 1 1) (thickness 0.15)) (justify mirror))
     )
@@
         (effects (font (size 1 1) (thickness 0.15)) (justify mirror))
     )
-    (fp_text value "CD74HC4067SM" (at 0 -5.64) (layer "B.Fab")
+    (fp_text value "CD74HC4067SM" (at 0 -5.64) (layer "B.Fab") hide
         (effects (font (size 1 1) (thickness 0.15)) (justify mirror))
     )
@@
         (effects (font (size 1 1) (thickness 0.15)) (justify mirror))
     )
-    (fp_text value "CD74HC4067SM" (at 0 5.83) (layer "B.Fab")
+    (fp_text value "CD74HC4067SM" (at 2.946 11.164 90) (layer "B.Fab")
         (effects (font (size 1 1) (thickness 0.15)) (justify mirror))
     )
@@
   (gr_line (start 151.000014 119.999986) (end 122.000014 119.999986)
     (stroke (width 0.05) (type solid)) (layer "Edge.Cuts"))
-  (gr_line (start 143.35 115.899) (end 150.15 115.899)
+  (gr_line (start 143.35 106.499) (end 150.15 106.499)
     (stroke (width 0.1) (type default)) (layer "B.Fab"))
-  (gr_text "Sensitive Sole v2.0\n" (at 130.404 127.508) (layer "B.SilkS")
-    (effects (font (size 1 1) (thickness 0.2) bold) (justify bottom))
-  )
-  (gr_text "Adrien Husson" (at 130.048 129.794) (layer "B.SilkS")
-    (effects (font (size 1 1) (thickness 0.125)) (justify bottom))
+  (gr_text "Sensitive Sole v2.0\n" (at 148.706 118.61) (layer "B.SilkS")
+    (effects (font (size 1 1) (thickness 0.2) bold) (justify left bottom mirror))
+  )
+  (gr_text "Adrn Hssn" (at 133.052 118.61) (layer "B.SilkS")
+    (effects (font (size 1 1) (thickness 0.125)) (justify left bottom mirror))
   )
   (dimension (type orthogonal) (layer "Dwgs.User")
@@
     (connect_pads (clearance 0.508))
     (min_thickness 0.25) (filled_areas_thickness no)
-    (fill yes (thermal_gap 0.5) (thermal_bridge_width 0.5))
+    (fill (thermal_gap 0.5) (thermal_bridge_width 0.5))
     (polygon
       (pts
@@
     (connect_pads (clearance 0.508))
     (min_thickness 0.25) (filled_areas_thickness no)
-    (fill yes (thermal_gap 0.5) (thermal_bridge_width 0.5))
+    (fill (thermal_gap 0.5) (thermal_bridge_width 0.5))
     (polygon
       (pts

Commit message: remove warnings
Parts:
- removed ? (x2): , 
- removed the REF** at (122.0, 118.0)
- added REF**: MountingHole_2.1mm, MountingHole:MountingHole_2.1mm, F.Cu at (122.0, 118.0)
- added REF**: MountingHole_2.1mm, MountingHole:MountingHole_2.1mm, F.Cu at (151.0, 118.0)
- added REF**: MountingHole_2.1mm, MountingHole:MountingHole_2.1mm, F.Cu at (151.0, 89.0)
- U$8: footprint MovuinoESP8266:LOGO-NoName_MOVUINO_BMP_11MM-TOP -> Movuino:LOGO-NoName_MOVUINO_BMP_11MM-TOP
Changed lines of the file:
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@@
   (net 69 "Net-(D1-DIN)")
   (net 70 "unconnected-(D1-DOUT-Pad4)")
-  (footprint "MountingHole:MountingHole_2.1mm" (layer "F.Cu")
-    (at 122.000014 117.999986)
-    (descr "Mounting Hole 2.1mm, no annular")
-    (tags "mounting hole 2.1mm no annular")
-    (attr exclude_from_pos_files exclude_from_bom)
-    (fp_text reference "REF**" (at -21.725905 -16.231425) (layer "F.SilkS") hide
-        (effects (font (size 1 1) (thickness 0.15)))
-    )
-    (fp_text value "MountingHole_2.1mm" (at -27.511619 -18.597965) (layer "F.Fab")
-        (effects (font (size 1 1) (thickness 0.15)))
-    )
-    (fp_text user "${REFERENCE}" (at -21.725905 -8.5) (layer "F.Fab")
-        (effects (font (size 1 1) (thickness 0.15)))
-    )
-    (fp_circle (center 0 0) (end 2.1 0)
-      (stroke (width 0.15) (type solid)) (fill none) (layer "Cmts.User"))
-    (fp_circle (center 0 0) (end 2.35 0)
-      (stroke (width 0.05) (type solid)) (fill none) (layer "F.CrtYd"))
-    (pad "" np_thru_hole circle (at 0 0) (size 2.1 2.1) (drill 2) (layers "*.Cu" "*.Mask"))
-  )
-  (footprint "MountingHole:MountingHole_2.1mm" (layer "F.Cu")
-    (at 122.000014 88.999986)
-    (descr "Mounting Hole 2.1mm, no annular")
-    (tags "mounting hole 2.1mm no annular")
-    (attr exclude_from_pos_files exclude_from_bom)
-    (fp_text reference "REF**" (at -21.725905 3.302415) (layer "F.SilkS") hide
-        (effects (font (size 1 1) (thickness 0.15)))
-    )
-    (fp_text value "MountingHole_2.1mm" (at -27.511619 5.668955) (layer "F.Fab")
-        (effects (font (size 1 1) (thickness 0.15)))
-    )
-    (fp_text user "${REFERENCE}" (at -21.725905 8.035495) (layer "F.Fab")
-        (effects (font (size 1 1) (thickness 0.15)))
-    )
-    (fp_circle (center 0 0) (end 2.1 0)
-      (stroke (width 0.15) (type solid)) (fill none) (layer "Cmts.User"))
-    (fp_circle (center 0 0) (end 2.35 0)
-      (stroke (width 0.05) (type solid)) (fill none) (layer "F.CrtYd"))
-    (pad "" np_thru_hole circle (at 0 0) (size 2.1 2.1) (drill 2) (layers "*.Cu" "B.Mask"))
-  )
-  (footprint "MovuinoESP8266:LOGO-NoName_MOVUINO_BMP_11MM-TOP" (layer "F.Cu")
+  (footprint "Movuino:LOGO-NoName_MOVUINO_BMP_11MM-TOP" (layer "F.Cu")
     (at 136.5 113.70632)
     (descr "Used parameters 0.007")
     (attr through_hole)
-    (fp_text reference "U$8" (at -35.551169 1.132745) (layer "F.SilkS") hide
-        (effects (font (size 1.27 1.27) (thickness 0.15)))
+    (fp_text reference "U$8" (at 0.42164 0.889) (layer "B.SilkS") hide
+        (effects (font (size 1.27 1.27) (thickness 0.15)) (justify mirror))
     )
-    (fp_text value "LOGO_MOVUINOBOTTOM_11MM" (at -47.676645 3.815185) (layer "F.SilkS") hide
+    (fp_text value "LOGO_MOVUINOBOTTOM_11MM" (at -21.8 -10.6 -180) (layer "F.SilkS") hide
         (effects (font (size 1.27 1.27) (thickness 0.15)))
     )
@@
       (stroke (width 0) (type solid)) (fill solid) (layer "F.SilkS"))
   )
+  (footprint "MountingHole:MountingHole_2.1mm" (layer "F.Cu")
+    (at 122.000014 118)
+    (descr "Mounting Hole 2.1mm, no annular")
+    (tags "mounting hole 2.1mm no annular")
+    (attr exclude_from_pos_files exclude_from_bom)
+    (fp_text reference "REF**" (at 0 -3.2) (layer "F.SilkS") hide
+        (effects (font (size 1 1) (thickness 0.15)))
+    )
+    (fp_text value "MountingHole_2.1mm" (at 0 3.2) (layer "F.Fab") hide
+        (effects (font (size 1 1) (thickness 0.15)))
+    )
+    (fp_text user "${REFERENCE}" (at 0 0) (layer "F.Fab") hide
+        (effects (font (size 1 1) (thickness 0.15)))
+    )
+    (fp_circle (center 0 0) (end 2.1 0)
+      (stroke (width 0.15) (type solid)) (fill none) (layer "Cmts.User"))
+    (fp_circle (center 0 0) (end 2.35 0)
+      (stroke (width 0.05) (type solid)) (fill none) (layer "F.CrtYd"))
+    (pad "" np_thru_hole circle (at 0 0) (size 2.1 2.1) (drill 2.1) (layers "F&B.Cu" "*.Mask"))
+  )
+  (footprint "MountingHole:MountingHole_2.1mm" (layer "F.Cu")
+    (at 151 118)
+    (descr "Mounting Hole 2.1mm, no annular")
+    (tags "mounting hole 2.1mm no annular")
+    (attr exclude_from_pos_files exclude_from_bom)
+    (fp_text reference "REF**" (at 0 -3.2) (layer "F.SilkS") hide
+        (effects (font (size 1 1) (thickness 0.15)))
+    )
+    (fp_text value "MountingHole_2.1mm" (at 0 3.2) (layer "F.Fab") hide
+        (effects (font (size 1 1) (thickness 0.15)))
+    )
+    (fp_text user "${REFERENCE}" (at 0 0) (layer "F.Fab") hide
+        (effects (font (size 1 1) (thickness 0.15)))
+    )
+    (fp_circle (center 0 0) (end 2.1 0)
+      (stroke (width 0.15) (type solid)) (fill none) (layer "Cmts.User"))
+    (fp_circle (center 0 0) (end 2.35 0)
+      (stroke (width 0.05) (type solid)) (fill none) (layer "F.CrtYd"))
+    (pad "" np_thru_hole circle (at 0 0) (size 2.1 2.1) (drill 2.1) (layers "F&B.Cu" "*.Mask"))
+  )
   (footprint "Connector_FFC-FPC:Molex_200528-0240_1x24-1MP_P1.00mm_Horizontal" (layer "F.Cu")
     (at 136.5 103.61)
@@
     (property "ki_keywords" "RGB LED NeoPixel addressable")
     (attr smd)
-    (fp_text reference "D1" (at 0 -3.5) (layer "F.SilkS") hide
+    (fp_text reference "D1" (at 0 -3.5 180) (layer "F.SilkS")
         (effects (font (size 1 1) (thickness 0.15)))
     )
-    (fp_text value "SK6812" (at 0 4) (layer "F.Fab") hide
+    (fp_text value "SK6812" (at 0 4 180) (layer "F.Fab")
         (effects (font (size 1 1) (thickness 0.15)))
     )
-    (fp_text user "${REFERENCE}" (at 0 0) (layer "F.Fab") hide
+    (fp_text user "${REFERENCE}" (at 0 0 180) (layer "F.Fab")
         (effects (font (size 0.8 0.8) (thickness 0.15)))
     )
+    (fp_line (start -3.65 -2.75) (end 3.65 -2.75)
+      (stroke (width 0.12) (type solid)) (layer "F.SilkS"))
+    (fp_line (start -3.65 2.75) (end 3.65 2.75)
+      (stroke (width 0.12) (type solid)) (layer "F.SilkS"))
+    (fp_line (start 3.65 2.75) (end 3.65 1.6)
+      (stroke (width 0.12) (type solid)) (layer "F.SilkS"))
     (fp_line (start -3.45 -2.75) (end -3.45 2.75)
       (stroke (width 0.05) (type solid)) (layer "F.CrtYd"))
@@
     )
   )
-  (footprint "" (layer "F.Cu")
-    (at 151.000014 117.999986)
-    (fp_text reference "" (at 0 0) (layer "F.SilkS")
-        (effects (font (size 1.27 1.27) (thickness 0.15)))
+  (footprint "MountingHole:MountingHole_2.1mm" (layer "F.Cu")
+    (at 151 88.999986)
+    (descr "Mounting Hole 2.1mm, no annular")
+    (tags "mounting hole 2.1mm no annular")
+    (attr exclude_from_pos_files exclude_from_bom)
+    (fp_text reference "REF**" (at 0 -3.2) (layer "F.SilkS") hide
+        (effects (font (size 1 1) (thickness 0.15)))
     )
-    (fp_text value "" (at 0 0) (layer "F.SilkS")
-        (effects (font (size 1.27 1.27) (thickness 0.15)))
+    (fp_text value "MountingHole_2.1mm" (at 0 3.2) (layer "F.Fab") hide
+        (effects (font (size 1 1) (thickness 0.15)))
+    )
+    (fp_text user "${REFERENCE}" (at 0 0) (layer "F.Fab") hide
+        (effects (font (size 1 1) (thickness 0.15)))
     )
-    (pad "" np_thru_hole circle (at 0 0) (size 2.1 2.1) (drill 2) (layers "*.Cu" "*.Mask"))
+    (fp_circle (center 0 0) (end 2.1 0)
+      (stroke (width 0.15) (type solid)) (fill none) (layer "Cmts.User"))
+    (fp_circle (center 0 0) (end 2.35 0)
+      (stroke (width 0.05) (type solid)) (fill none) (layer "F.CrtYd"))
+    (pad "" np_thru_hole circle (at 0 0) (size 2.1 2.1) (drill 2.1) (layers "F&B.Cu" "*.Mask"))
   )
-  (footprint "" (layer "F.Cu")
+  (footprint "MountingHole:MountingHole_2.1mm" (layer "F.Cu")
     (at 122.000014 88.999986)
-    (fp_text reference "" (at 0 0) (layer "F.SilkS")
-        (effects (font (size 1.27 1.27) (thickness 0.15)))
+    (descr "Mounting Hole 2.1mm, no annular")
+    (tags "mounting hole 2.1mm no annular")
+    (attr exclude_from_pos_files exclude_from_bom)
+    (fp_text reference "REF**" (at 0 -3.2) (layer "F.SilkS") hide
+        (effects (font (size 1 1) (thickness 0.15)))
     )
-    (fp_text value "" (at 0 0) (layer "F.SilkS")
-        (effects (font (size 1.27 1.27) (thickness 0.15)))
+    (fp_text value "MountingHole_2.1mm" (at 0 3.2) (layer "F.Fab") hide
+        (effects (font (size 1 1) (thickness 0.15)))
+    )
+    (fp_text user "${REFERENCE}" (at 0 0) (layer "F.Fab") hide
+        (effects (font (size 1 1) (thickness 0.15)))
     )
-    (pad "" np_thru_hole circle (at 29 0) (size 2.1 2.1) (drill 2) (layers "*.Cu" "B.Mask"))
+    (fp_circle (center 0 0) (end 2.1 0)
+      (stroke (width 0.15) (type solid)) (fill none) (layer "Cmts.User"))
+    (fp_circle (center 0 0) (end 2.35 0)
+      (stroke (width 0.05) (type solid)) (fill none) (layer "F.CrtYd"))
+    (pad "" np_thru_hole circle (at 0 0) (size 2.1 2.1) (drill 2.1) (layers "*.Cu" "*.Mask"))
   )
   (footprint "Movuino:DF12-36-DP-NL" (layer "B.Cu")
@@
     (height -8.414214)
     (orientation 1)
-    (gr_text "17,8000 mm" (at 111.7858 111.099993 90) (layer "Dwgs.User")
+    (gr_text "17.8000 mm" (at 111.7858 111.099993 90) (layer "Dwgs.User")
       (effects (font (size 1.5 1.5) (thickness 0.3)))
     )
@@
     (height 9.585786)
     (orientation 1)
-    (gr_text "33,0000 mm" (at 158.7858 103.499986 90) (layer "Dwgs.User")
+    (gr_text "33.0000 mm" (at 158.7858 103.499986 90) (layer "Dwgs.User")
       (effects (font (size 1.5 1.5) (thickness 0.3)))
     )
@@
     (connect_pads (clearance 0.508))
     (min_thickness 0.25) (filled_areas_thickness no)
-    (fill (thermal_gap 0.5) (thermal_bridge_width 0.5))
+    (fill yes (thermal_gap 0.5) (thermal_bridge_width 0.5))
     (polygon
       (pts
@@
     (connect_pads (clearance 0.508))
     (min_thickness 0.25) (filled_areas_thickness no)
-    (fill (thermal_gap 0.5) (thermal_bridge_width 0.5))
+    (fill yes (thermal_gap 0.5) (thermal_bridge_width 0.5))
     (polygon
       (pts
