File: SensitiveSole.kicad_pcb (KiCad board)
At the start: 2 copper layers, 33 x 33 mm, 21 parts

Commit message: ready to order
Parts:
- D1: value SK6812 -> WS2812B; footprint LED_SMD:LED_SK6812_PLCC4_5.0x5.0mm_P3.2mm -> LED_SMD:LED_WS2812B_PLCC4_5.0x5.0mm_P3.2mm
- R8: value 470 -> 470Ω
- turned D1 to 0 degrees
Routing:
- net /IO26: track 24.2 -> 23.2 mm
Changed lines of the file:
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@@
     )
   )
-  (footprint "LED_SMD:LED_SK6812_PLCC4_5.0x5.0mm_P3.2mm" (layer "F.Cu")
-    (at 136.5 94.35 180)
-    (descr "5.0mm x 5.0mm Addressable RGB LED NeoPixel, https://cdn-shop.adafruit.com/product-files/1138/SK6812+LED+datasheet+.pdf")
+  (footprint "LED_SMD:LED_WS2812B_PLCC4_5.0x5.0mm_P3.2mm" (layer "F.Cu")
+    (at 136.5 94.35)
+    (descr "5.0mm x 5.0mm Addressable RGB LED NeoPixel, https://cdn-shop.adafruit.com/datasheets/WS2812B.pdf")
     (tags "LED RGB NeoPixel PLCC-4 5050")
     (property "Sheetfile" "SensitiveSole.kicad_sch")
@@
     (property "ki_keywords" "RGB LED NeoPixel addressable")
     (attr smd)
-    (fp_text reference "D1" (at 0 -3.5 180) (layer "F.SilkS")
+    (fp_text reference "D1" (at 0 -3.5) (layer "F.SilkS") hide
         (effects (font (size 1 1) (thickness 0.15)))
     )
-    (fp_text value "SK6812" (at 0 4 180) (layer "F.Fab")
+    (fp_text value "WS2812B" (at 0 4) (layer "F.Fab") hide
         (effects (font (size 1 1) (thickness 0.15)))
     )
-    (fp_text user "${REFERENCE}" (at 0 0 180) (layer "F.Fab")
+    (fp_text user "1" (at -4.15 -1.6) (layer "F.SilkS") hide
+        (effects (font (size 1 1) (thickness 0.15)))
+    )
+    (fp_text user "${REFERENCE}" (at 0 0) (layer "F.Fab") hide
         (effects (font (size 0.8 0.8) (thickness 0.15)))
     )
-    (fp_line (start -3.65 -2.75) (end 3.65 -2.75)
-      (stroke (width 0.12) (type solid)) (layer "F.SilkS"))
-    (fp_line (start -3.65 2.75) (end 3.65 2.75)
-      (stroke (width 0.12) (type solid)) (layer "F.SilkS"))
-    (fp_line (start 3.65 2.75) (end 3.65 1.6)
-      (stroke (width 0.12) (type solid)) (layer "F.SilkS"))
     (fp_line (start -3.45 -2.75) (end -3.45 2.75)
       (stroke (width 0.05) (type solid)) (layer "F.CrtYd"))
@@
     (fp_circle (center 0 0) (end 0 -2)
       (stroke (width 0.1) (type solid)) (fill none) (layer "F.Fab"))
-    (pad "1" smd rect (at 2.45 1.6 180) (size 1.5 1) (layers "F.Cu" "F.Paste" "F.Mask")
+    (pad "1" smd rect (at -2.45 -1.65) (size 1.5 0.9) (layers "F.Cu" "F.Paste" "F.Mask")
       (net 1 "GND") (pinfunction "VSS") (pintype "power_in"))
-    (pad "2" smd rect (at 2.45 -1.6 180) (size 1.5 1) (layers "F.Cu" "F.Paste" "F.Mask")
+    (pad "2" smd rect (at -2.45 1.65) (size 1.5 0.9) (layers "F.Cu" "F.Paste" "F.Mask")
       (net 69 "Net-(D1-DIN)") (pinfunction "DIN") (pintype "input"))
-    (pad "3" smd rect (at -2.45 -1.6 180) (size 1.5 1) (layers "F.Cu" "F.Paste" "F.Mask")
+    (pad "3" smd rect (at 2.45 1.65) (size 1.5 0.9) (layers "F.Cu" "F.Paste" "F.Mask")
       (net 68 "Net-(D1-VDD)") (pinfunction "VDD") (pintype "power_in"))
-    (pad "4" smd rect (at -2.45 1.6 180) (size 1.5 1) (layers "F.Cu" "F.Paste" "F.Mask")
+    (pad "4" smd rect (at 2.45 -1.65) (size 1.5 0.9) (layers "F.Cu" "F.Paste" "F.Mask")
       (net 70 "unconnected-(D1-DOUT-Pad4)") (pinfunction "DOUT") (pintype "output"))
-    (model "${KICAD7_3DMODEL_DIR}/LED_SMD.3dshapes/LED_SK6812_PLCC4_5.0x5.0mm_P3.2mm.wrl"
+    (model "${KICAD7_3DMODEL_DIR}/LED_SMD.3dshapes/LED_WS2812B_PLCC4_5.0x5.0mm_P3.2mm.wrl"
       (offset (xyz 0 0 0))
       (scale (xyz 1 1 1))
@@
         (effects (font (size 1 1) (thickness 0.15)) (justify mirror))
     )
-    (fp_text value "10µ" (at 0.0265 -1.524 90) (layer "B.Fab")
+    (fp_text value "10µ" (at 0.0265 -1.674 90) (layer "B.SilkS")
         (effects (font (size 1 1) (thickness 0.15)) (justify mirror))
     )
@@
         (effects (font (size 1 1) (thickness 0.15)) (justify mirror))
     )
-    (fp_text value "0.1µ" (at 0.0265 -1.462 90) (layer "B.Fab")
+    (fp_text value "0.1µ" (at 0.0265 -1.612 90) (layer "B.SilkS")
         (effects (font (size 1 1) (thickness 0.15)) (justify mirror))
     )
@@
         (effects (font (size 1 1) (thickness 0.15)) (justify mirror))
     )
-    (fp_text value "10kΩ" (at -1.558 9.11) (layer "B.Fab")
+    (fp_text value "10kΩ" (at -1.558 9.11) (layer "B.SilkS")
         (effects (font (size 1 1) (thickness 0.15)) (justify mirror))
     )
@@
         (effects (font (size 1 1) (thickness 0.15)) (justify mirror))
     )
-    (fp_text value "0.1µ" (at 0 -1.678 90) (layer "B.Fab")
+    (fp_text value "0.1µ" (at 0 -1.878 90) (layer "B.SilkS")
         (effects (font (size 1 1) (thickness 0.15)) (justify mirror))
     )
@@
     (property "ki_keywords" "R res resistor")
     (attr smd)
-    (fp_text reference "R8" (at 0 1.43) (layer "B.SilkS")
-        (effects (font (size 1 1) (thickness 0.15)) (justify mirror))
-    )
-    (fp_text value "470" (at 0 -1.43) (layer "B.Fab")
-        (effects (font (size 1 1) (thickness 0.15)) (justify mirror))
-    )
-    (fp_text user "${REFERENCE}" (at 0 0) (layer "B.Fab")
+    (fp_text reference "R8" (at 0 1.43) (layer "B.SilkS") hide
+        (effects (font (size 1 1) (thickness 0.15)) (justify mirror))
+    )
+    (fp_text value "470Ω" (at 0 -1.43) (layer "B.SilkS")
+        (effects (font (size 1 1) (thickness 0.15)) (justify mirror))
+    )
+    (fp_text user "${REFERENCE}" (at 0 0) (layer "B.Fab") hide
         (effects (font (size 0.4 0.4) (thickness 0.06)) (justify mirror))
     )
@@
         (effects (font (size 1 1) (thickness 0.15)) (justify mirror))
     )
-    (fp_text value "CD74HC4067SM" (at 2.946 11.164 90) (layer "B.Fab")
+    (fp_text value "CD74HC4067SM" (at 2.946 11.164 90) (layer "B.SilkS")
         (effects (font (size 1 1) (thickness 0.15)) (justify mirror))
     )
@@
     )
   )
+  (gr_line (start 143.35 106.499) (end 150.15 106.499)
+    (stroke (width 0.1) (type default)) (layer "B.SilkS"))
   (gr_curve (pts (xy 127.715078 94.35) (xy 127.715078 91.671546) (xy 131.630269 89.508462) (xy 136.500001 89.508462))
     (stroke (width 0.18) (type solid)) (layer "F.SilkS"))
@@
   (gr_line (start 151.000014 119.999986) (end 122.000014 119.999986)
     (stroke (width 0.05) (type solid)) (layer "Edge.Cuts"))
-  (gr_line (start 143.35 106.499) (end 150.15 106.499)
-    (stroke (width 0.1) (type default)) (layer "B.Fab"))
   (gr_text "Sensitive Sole v2.0\n" (at 148.706 118.61) (layer "B.SilkS")
     (effects (font (size 1 1) (thickness 0.2) bold) (justify left bottom mirror))
@@
   (segment (start 133.561396 114.425) (end 129.9 114.425) (width 0.25) (layer "B.Cu") (net 17))
   (segment (start 131.409986 103.249986) (end 134.55 106.39) (width 0.25) (layer "B.Cu") (net 17))
-  (segment (start 131.27359 103.749986) (end 132.31 104.786396) (width 0.25) (layer "B.Cu") (net 19))
-  (segment (start 127.87 106.172) (end 127.87 115.075) (width 0.25) (layer "B.Cu") (net 19))
-  (segment (start 127.87 115.075) (end 129.9 115.075) (width 0.25) (layer "B.Cu") (net 19))
-  (segment (start 132.31 106.172) (end 127.87 106.172) (width 0.25) (layer "B.Cu") (net 19))
-  (segment (start 132.31 104.786396) (end 132.31 106.172) (width 0.25) (layer "B.Cu") (net 19))
-  (segment (start 125.300114 103.749986) (end 131.27359 103.749986) (width 0.25) (layer "B.Cu") (net 19))
+  (segment (start 131.464557 103.940953) (end 132.119034 104.59543) (width 0.25) (layer "B.Cu") (net 19))
+  (segment (start 127.87 106.824) (end 127.87 114.423) (width 0.25) (layer "B.Cu") (net 19))
+  (segment (start 128.522 115.075) (end 129.9 115.075) (width 0.25) (layer "B.Cu") (net 19))
+  (segment (start 131.658 106.172) (end 128.522 106.172) (width 0.25) (layer "B.Cu") (net 19))
+  (segment (start 132.31 105.056463) (end 132.31 105.52) (width 0.25) (layer "B.Cu") (net 19))
+  (segment (start 125.300114 103.749986) (end 131.003523 103.749986) (width 0.25) (layer "B.Cu") (net 19))
+  (arc (start 132.119034 104.59543) (mid 132.260369 104.806954) (end 132.31 105.056463) (width 0.25) (layer "B.Cu") (net 19))
+  (arc (start 127.87 114.423) (mid 128.060966 114.884034) (end 128.522 115.075) (width 0.25) (layer "B.Cu") (net 19))
+  (arc (start 131.658 106.172) (mid 132.119034 105.981034) (end 132.31 105.52) (width 0.25) (layer "B.Cu") (net 19))
+  (arc (start 127.87 106.824) (mid 128.060966 106.362966) (end 128.522 106.172) (width 0.25) (layer "B.Cu") (net 19))
+  (arc (start 131.464557 103.940953) (mid 131.253033 103.799617) (end 131.003523 103.749986) (width 0.25) (layer "B.Cu") (net 19))
   (segment (start 124.054 104.103872) (end 124.054 94.175) (width 0.2) (layer "B.Cu") (net 21))
   (segment (start 125.300114 104.249986) (end 124.200114 104.249986) (width 0.2) (layer "B.Cu") (net 21))
