File: SensitiveSole.kicad_sch (KiCad schematic)
At the start: 13 parts, among them U1 CD74HC4067SM, U2 CD74HC4067SM

Commit message: doc
Connections:
- net GND: now also U1.16 (I15), U1.17 (I14), U1.18 (I13), U1.19 (I12), U1.2 (I7), U1.20 (I11), U1.21 (I10), U1.22 (I9), U1.23 (I8), U2.16 (I15)
Other:
- note added: "A1 ADC1_CH2 GPI38"
- note added: "A2 ADC1_CH3 GPI39"
- note added: "A3 ADC1_CH6 GPI34"
- note added: "A4 ADC1_CH1 GPI37"
- note added: "A5 ADC1_CH7 GPI35"
- note added: "BATT Monitoring (A0 ADC1_CH0) GPI36"
- note added: "BUILTIN NEOPIXEL (TOUCH3 D6 ADC2_CH3) GPIO15"
- note added: "DAC_1 D2 ADC2_CH8 GPIO25"
- note added: "DAC_2 D3 ADC2_CH9 GPIO26"
- note added: "INPUT ONLY"
- note added: "INT BUILTIN MPU (TOUCH0 D9 ADC2_CH0) GPIO4"
- note added: "PB_OUT (TOUCH4 D8 ADC2_CH4) GPIO13"
- note added: "PS_HOLD (TOUCH5 D7 ADC2_CH5) GPIO12"
- note added: "TOUCH2 X2 ADC2_CH2 GPIO2"
- note added: "TOUCH6 D5 ADC2_CH6 GPIO14"
- note added: "TOUCH7 D4 ADC2_CH7 GPIO27"
- note added: "TOUCH8 D1 ADC1_CH5 GPIO33"
- note added: "TOUCH9 A6 ADC1_CH4 GPIO32"
- note removed: "A1 ADC1_CH2"
- note removed: "A2 ADC1_CH3"
- note removed: "A3 ADC1_CH6"
- note removed: "A4 ADC1_CH1"
- note removed: "A5 ADC1_CH7"
- note removed: "BATT Monitoring (A0 ADC1_CH0)"
- note removed: "BUILTIN NEOPIXEL (TOUCH3 D6 ADC2_CH3)"
- note removed: "DAC_1 D2 ADC2_CH8"
- note removed: "DAC_2 D3 ADC2_CH9"
- note removed: "INT BUILTIN MPU (TOUCH0 D9 ADC2_CH0)"
- note removed: "PB_OUT (TOUCH4 D8 ADC2_CH4)"
- note removed: "PS_HOLD (TOUCH5 D7 ADC2_CH5)"
- note removed: "TOUCH2 X2 ADC2_CH2"
- note removed: "TOUCH6 D5 ADC2_CH6"
- note removed: "TOUCH7 D4 ADC2_CH7"
- note removed: "TOUCH8 D1 ADC1_CH5"
- note removed: "TOUCH9 A6 ADC1_CH4"

Commit message: base clean
Parts:
- renumbered FPC to FPC1
Connections:
- net GND: no longer U1.16 (I15), U1.17 (I14), U1.18 (I13), U1.19 (I12), U1.2 (I7), U1.20 (I11), U1.21 (I10), U1.22 (I9), U1.23 (I8), U2.16 (I15)
- net IO12: now also U2.14 (S2); no longer U2.1 (COM)
- net IO14: now also U2.11 (S1); no longer U2.13 (S3)
- net IO25: now also U1.14 (S2); no longer U1.1 (COM)
- net IO26: now also U1.13 (S3); no longer U1.14 (S2)
- net IO27: now also U2.10 (S0); no longer U1.13 (S3)
- net IO32: now also U1.10 (S0); no longer U1.11 (S1)
- net IO33: now also U1.11 (S1); no longer U1.10 (S0)
- net IO39: now also U1.1 (COM)
- net IO5: now also U2.13 (S3)
- net GPIO2 renamed IO2
- net IO2: now also U2.1 (COM)
- net IO13: no longer names the net of BOTTOM_DF12.29
- net IO13: no longer U2.10 (S0)
- net IO15: no longer names the net of BOTTOM_DF12.25
- net IO15: no longer U2.14 (S2)
- net IO34: no longer names the net of BOTTOM_DF12.7
- net IO35: no longer names the net of BOTTOM_DF12.11
- net IO37: no longer names the net of BOTTOM_DF12.9
- net IO38: no longer names the net of BOTTOM_DF12.3
- net IO4: no longer names the net of BOTTOM_DF12.31
- net IO4: no longer U2.11 (S1)
Other:
- note removed: "INT BUILTIN MPU (TOUCH0 D9 ADC2_CH0) GPIO4"
- note removed: "PB_OUT (TOUCH4 D8 ADC2_CH4) GPIO13"
- moved on the sheet: BOTTOM_DF12, C1, C2, FPC1, U1, U2

Commit message: v0.99
Parts:
- added C3: 0.1µ, Capacitor_SMD:C_0603_1608Metric_Pad1.08x0.95mm_HandSolder, symbol Device:C
- added D1: SK6812, LED_SMD:LED_SK6812_PLCC4_5.0x5.0mm_P3.2mm, symbol LED:SK6812
- added R8: 470, Resistor_SMD:R_0603_1608Metric_Pad0.98x0.95mm_HandSolder, symbol Device:R
Connections:
- net +3.3V: now also C3.1
- net GND: now also D1.1 (VSS)
- net IO15: now reaches BOTTOM_DF12.25
- net IO15: now also R8.1
- new net: D1.2 (DIN), R8.2
- new net: C3.2, D1.3 (VDD)
Changed lines of the file:
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@@
+    (stroke (width 0) (type default))
+  )
+  (wire (pts (xy 80.01 153.67) (xy 86.36 153.67))
     (stroke (width 0) (type default))
   )
@@
     (effects (font (size 1.27 1.27)) (justify right bottom))
   )
+  (label "IO15" (at 85.09 62.23 180) (fields_autoplaced)
+    (effects (font (size 1.27 1.27)) (justify right bottom))
+  )
   (label "ROW8" (at 250.19 60.96 180) (fields_autoplaced)
     (effects (font (size 1.27 1.27)) (justify right bottom))
@@
   (label "ROW10" (at 199.39 60.96 0) (fields_autoplaced)
     (effects (font (size 1.27 1.27)) (justify left bottom))
+  )
+  (label "IO15" (at 80.01 153.67 180) (fields_autoplaced)
+    (effects (font (size 1.27 1.27)) (justify right bottom))
   )
   (label "ROW2" (at 199.39 40.64 0) (fields_autoplaced)
@@
     )
   )
+  (symbol (lib_id "LED:SK6812") (at 101.6 153.67 0) (unit 1)
+    (in_bom yes) (on_board yes) (dnp no)
+    (property "Reference" "D1" (at 113.03 154.94 0)
+      (effects (font (size 1.27 1.27)))
+    )
+    (property "Value" "SK6812" (at 111.76 157.48 0)
+      (effects (font (size 1.27 1.27)))
+    )
+    (property "Footprint" "LED_SMD:LED_SK6812_PLCC4_5.0x5.0mm_P3.2mm" (at 102.87 161.29 0)
+      (effects (font (size 1.27 1.27)) (justify left top) hide)
+    )
+    (property "Datasheet" "https://cdn-shop.adafruit.com/product-files/1138/SK6812+LED+datasheet+.pdf" (at 104.14 163.195 0)
+      (effects (font (size 1.27 1.27)) (justify left top) hide)
+    )
+    (pin "1")
+    (pin "3")
+    (pin "4")
+    (pin "2")
+    (instances
+      (project "SensitiveSole"
+        (path "/f67b8ac4-d503-4876-8468-34a7f8dc7022"
+          (reference "D1") (unit 1)
+        )
+      )
+    )
+  )
+  (symbol (lib_id "power:GND") (at 101.6 161.29 0) (unit 1)
+    (in_bom yes) (on_board yes) (dnp no) (fields_autoplaced)
+    (property "Reference" "#PWR016" (at 101.6 167.64 0)
+      (effects (font (size 1.27 1.27)) hide)
+    )
+    (property "Value" "GND" (at 101.6 166.37 0)
+      (effects (font (size 1.27 1.27)))
+    )
+    (property "Footprint" "" (at 101.6 161.29 0)
+      (effects (font (size 1.27 1.27)) hide)
+    )
+    (property "Datasheet" "" (at 101.6 161.29 0)
+      (effects (font (size 1.27 1.27)) hide)
+    )
+    (pin "1")
+    (instances
+      (project "SensitiveSole"
+        (path "/f67b8ac4-d503-4876-8468-34a7f8dc7022"
+          (reference "#PWR016") (unit 1)
+        )
+      )
+    )
+  )
   (symbol (lib_id "power:GND") (at 177.8 81.28 0) (unit 1)
     (in_bom yes) (on_board yes) (dnp no) (fields_autoplaced)
@@
         (path "/f67b8ac4-d503-4876-8468-34a7f8dc7022"
           (reference "#PWR02") (unit 1)
+        )
+      )
+    )
+  )
+  (symbol (lib_id "Device:R") (at 90.17 153.67 90) (unit 1)
+    (in_bom yes) (on_board yes) (dnp no)
+    (property "Reference" "R8" (at 90.17 147.32 90)
+      (effects (font (size 1.27 1.27)) hide)
+    )
+    (property "Value" "470" (at 90.17 151.13 90)
+      (effects (font (size 1.27 1.27)))
+    )
+    (property "Footprint" "Resistor_SMD:R_0603_1608Metric_Pad0.98x0.95mm_HandSolder" (at 90.17 155.448 90)
+      (effects (font (size 1.27 1.27)) hide)
+    )
+    (property "Datasheet" "~" (at 90.17 153.67 0)
+      (effects (font (size 1.27 1.27)) hide)
+    )
+    (pin "1")
+    (pin "2")
+    (instances
+      (project "SensitiveSole"
+        (path "/f67b8ac4-d503-4876-8468-34a7f8dc7022"
+          (reference "R8") (unit 1)
+        )
+      )
+    )
+  )
+  (symbol (lib_id "power:+3.3V") (at 101.6 138.43 0) (unit 1)
+    (in_bom yes) (on_board yes) (dnp no) (fields_autoplaced)
+    (property "Reference" "#PWR017" (at 101.6 142.24 0)
+      (effects (font (size 1.27 1.27)) hide)
+    )
+    (property "Value" "+3.3V" (at 101.6 133.35 0)
+      (effects (font (size 1.27 1.27)))
+    )
+    (property "Footprint" "" (at 101.6 138.43 0)
+      (effects (font (size 1.27 1.27)) hide)
+    )
+    (property "Datasheet" "" (at 101.6 138.43 0)
+      (effects (font (size 1.27 1.27)) hide)
+    )
+    (pin "1")
+    (instances
+      (project "SensitiveSole"
+        (path "/f67b8ac4-d503-4876-8468-34a7f8dc7022"
+          (reference "#PWR017") (unit 1)
         )
       )
@@
         )
       )
+    )
+  )
+  (symbol (lib_id "Device:C") (at 101.6 142.24 0) (unit 1)
+    (in_bom yes) (on_board yes) (dnp no) (fields_autoplaced)
+    (property "Reference" "C3" (at 105.41 140.97 0)
+      (effects (font (size 1.27 1.27)) (justify left))
+    )
+    (property "Value" "0.1µ" (at 105.41 143.51 0)
+      (effects (font (size 1.27 1.27)) (justify left))
+    )
+    (property "Footprint" "Capacitor_SMD:C_0603_1608Metric_Pad1.08x0.95mm_HandSolder" (at 102.5652 146.05 0)
+      (effects (font (size 1.27 1.27)) hide)
+    )
+    (property "Datasheet" "~" (at 101.6 142.24 0)
+      (effects (font (size 1.27 1.27)) hide)
+    )
+    (pin "1")
+    (pin "2")
+    (instances
+      (project "SensitiveSole"
+        (path "/f67b8ac4-d503-4876-8468-34a7f8dc7022"
+          (reference "C3") (unit 1)
+        )
+      )

Commit message: graphism
Parts:
- BOTTOM_DF12: footprint MovuinoESP8266:DF12-36-DP-NL -> Movuino:DF12-36-DP-NL
Changed lines of the file:
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@@
       (effects (font (size 1.4986 1.4986)))
     )
-    (property "Footprint" "MovuinoESP8266:DF12-36-DP-NL" (at 104.14 49.53 0)
+    (property "Footprint" "Movuino:DF12-36-DP-NL" (at 104.14 49.53 0)
       (effects (font (size 1.27 1.27)) hide)
     )

Commit message: ready to order
Parts:
- D1: value SK6812 -> WS2812B; footprint LED_SMD:LED_SK6812_PLCC4_5.0x5.0mm_P3.2mm -> LED_SMD:LED_WS2812B_PLCC4_5.0x5.0mm_P3.2mm
Changed lines of the file:
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@@
       (effects (font (size 1.27 1.27)))
     )
-    (property "Value" "SK6812" (at 111.76 157.48 0)
+    (property "Value" "WS2812B" (at 111.76 157.48 0)
       (effects (font (size 1.27 1.27)))
     )
-    (property "Footprint" "LED_SMD:LED_SK6812_PLCC4_5.0x5.0mm_P3.2mm" (at 102.87 161.29 0)
+    (property "Footprint" "LED_SMD:LED_WS2812B_PLCC4_5.0x5.0mm_P3.2mm" (at 102.87 161.29 0)
       (effects (font (size 1.27 1.27)) (justify left top) hide)
     )
@@
     )
     (pin "1")
+    (pin "2")
     (pin "3")
     (pin "4")
-    (pin "2")
     (instances
       (project "SensitiveSole"
